File: pumpkin.kicad_pcb (KiCad board)
At the start: 2 copper layers, 92.9 x 79.5 mm, 3 parts

Commit message: add pumpkin art
Parts:
- added REF**: LED_0805_2012Metric_Pad1.15x1.40mm_HandSolder, afterdark:LED_0805_2012Metric_Pad1.15x1.40mm_HandSolder, F.Cu at (174.0, 61.2)
- added V: HOLE-PLATED-200MIL, afterdark:HOLE-UNPLATED, F.Cu at (170.0, 71.4)
Changed lines of the file:
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@@
       (outputformat 1)
       (mirror false)
-      (drillshape 1)
+      (drillshape 0)
       (scaleselection 1)
-      (outputdirectory "")
+      (outputdirectory "gerbers/pumpkin-v1")
     )
   )
   (net 0 "")
+  (module "afterdark:LED_0805_2012Metric_Pad1.15x1.40mm_HandSolder" (layer "F.Cu")
+    (at 174.0408 61.1632)
+    (descr "LED SMD 0805 (2012 Metric), square (rectangular) end terminal, IPC_7351 nominal, (Body size source: https://docs.google.com/spreadsheets/d/1BsfQQcO9C6DZCsRaXUlFlo91Tg2WpOkGARC1WS5S8t0/edit?usp=sharing), generated with kicad-footprint-generator")
+    (tags "LED handsolder")
+    (attr smd)
+    (fp_text reference "REF**" (at 0 -1.65 -180) (layer "F.SilkS") hide
+      (effects (font (size 1 1) (thickness 0.15)))
+    )
+    (fp_text value "LED_0805_2012Metric_Pad1.15x1.40mm_HandSolder" (at 0 1.65 -180) (layer "F.Fab") hide
+      (effects (font (size 1 1) (thickness 0.15)))
+    )
+    (fp_text user "+" (at -2.3114 -1.3462) (layer "F.SilkS")
+      (effects (font (size 1 1) (thickness 0.15)))
+    )
+    (fp_text user "${REFERENCE}" (at 0 0 -180) (layer "F.Fab") hide
+      (effects (font (size 0.5 0.5) (thickness 0.08)))
+    )
+    (fp_line (start -1.85 -0.95) (end 1.85 -0.95) (layer "F.CrtYd") (width 0.05))
+    (fp_line (start 1.85 -0.95) (end 1.85 0.95) (layer "F.CrtYd") (width 0.05))
+    (fp_line (start 1.85 0.95) (end -1.85 0.95) (layer "F.CrtYd") (width 0.05))
+    (fp_line (start -1.85 0.95) (end -1.85 -0.95) (layer "F.CrtYd") (width 0.05))
+    (fp_line (start 1 0.6) (end 1 -0.6) (layer "F.Fab") (width 0.1))
+    (fp_line (start 1 -0.6) (end -0.7 -0.6) (layer "F.Fab") (width 0.1))
+    (fp_line (start -1 0.6) (end 1 0.6) (layer "F.Fab") (width 0.1))
+    (fp_line (start -0.7 -0.6) (end -1 -0.3) (layer "F.Fab") (width 0.1))
+    (fp_line (start -1 -0.3) (end -1 0.6) (layer "F.Fab") (width 0.1))
+    (pad "1" smd roundrect (at -1.025 0) (size 1.15 1.4) (layers "F.Cu" "F.Paste" "F.Mask") (roundrect_rratio 0.217391))
+    (pad "2" smd roundrect (at 1.025 0) (size 1.15 1.4) (layers "F.Cu" "F.Paste" "F.Mask") (roundrect_rratio 0.217391))
+    (model "${KISYS3DMOD}/LED_SMD.3dshapes/LED_0805_2012Metric.wrl"
+      (offset (xyz 0 0 0))
+      (scale (xyz 1 1 1))
+      (rotate (xyz 0 0 0))
+    )
+  )
   (module "art:pumpkin-neg" (layer "F.Cu")
     (at 171.704 102.2604)
@@
       (xy -15.131316 -30.535965)) (layer "F.Cu") (width 0.01))
   )
+  (module "afterdark:HOLE-UNPLATED" (layer "F.Cu")
+    (at 170.01744 71.39432)
+    (attr exclude_from_pos_files exclude_from_bom)
+    (fp_text reference "V" (at 0 -2) (layer "F.SilkS") hide
+      (effects (font (size 1.016 1.016) (thickness 0.1524)))
+    )
+    (fp_text value "HOLE-PLATED-200MIL" (at -2.1 2.88 90) (layer "F.Fab") hide
+      (effects (font (size 1 1) (thickness 0.15)))
+    )
+    (pad "" np_thru_hole circle (at 0.94996 1.19888) (size 2.54 2.54) (drill 2.54) (layers *.Mask))
+  )
   (module "art:pumpkin-outline" (layer "F.Cu")
     (at 170.959492 101.28765)
@@
   )
   (gr_poly (pts
- (xy 233.377734 149.776922)
-    (xy 178.640419 148.975888)
-    (xy 122.568048 142.834629)
-    (xy 98.804043 57.391016)
-    (xy 106.814382 44.841485)
-    (xy 216.823034 44.307462)) (layer "B.Mask") (width 0.1))
+ (xy 81.805283 117.0686)
+    (xy -61.8998 117.0686)
+    (xy -61.8998 7.393537)
+    (xy 81.805283 7.393537)) (layer "B.Mask") (width 0.1))
   (gr_poly (pts
- (xy 181.88846 59.248677)
-    (xy 181.267477 61.235822)
-    (xy 176.548007 66.017391)
-    (xy 175.989122 71.668336)
-    (xy 175.989122 72.289319)
-    (xy 175.573191 72.850827)
-    (xy 172.328922 73.724283)
-    (xy 170.893957 74.015436)
-    (xy 167.153598 72.84095)
-    (xy 166.981955 72.482586)
-    (xy 168.102639 62.539887)
-    (xy 171.952733 56.95104)
-    (xy 173.939879 55.895369)) (layer "F.Mask") (width 0.1))
+ (xy 50.601127 150.989237)
+    (xy 49.980144 152.976382)
+    (xy 45.260674 157.757951)
+    (xy 44.701789 163.408896)
+    (xy 44.701789 164.029879)
+    (xy 44.285858 164.591387)
+    (xy 41.041589 165.464843)
+    (xy 39.606624 165.755996)
+    (xy 35.866265 164.58151)
+    (xy 35.694622 164.223146)
+    (xy 36.815306 154.280447)
+    (xy 40.6654 148.6916)
+    (xy 42.652546 147.635929)) (layer "F.Mask") (width 0.1))
 )
