File: art3.kicad_pcb (KiCad board)
At the start: 2 copper layers, 221.6 x 124.9 mm, 2 parts

Commit message: add pumpkin art and improved blm keychain
Routing:
- net (no net): track 52.6 -> 53.7 mm
Changed lines of the file:
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@@
-(kicad_pcb (version 20200922) (generator pcbnew)
+(kicad_pcb (version 20201002) (generator pcbnew)
   (general
     (thickness 1.6)
@@
   )
   (gr_rect (start 41.148 37.084) (end 262.7376 162.0012) (layer "Edge.Cuts") (width 0.05))
-  (segment (start 112.296406 71.55545) (end 112.884428 71.482924) (width 0.25) (layer "F.Cu") (net 0))
-  (segment (start 112.884428 71.482924) (end 113.4753 71.439339) (width 0.25) (layer "F.Cu") (net 0))
-  (segment (start 131.6848 74.7014) (end 131.9205 74.9371) (width 0.25) (layer "F.Cu") (net 0))
-  (segment (start 107.361273 73.45914) (end 107.86183 73.142166) (width 0.25) (layer "F.Cu") (net 0))
-  (segment (start 105.961166 74.551795) (end 106.409795 74.164805) (width 0.25) (layer "F.Cu") (net 0))
-  (segment (start 132.777 75.7936) (end 132.9111 75.9277) (width 0.25) (layer "F.Cu") (net 0))
-  (segment (start 108.377337 72.850135) (end 108.906553 72.58375) (width 0.25) (layer "F.Cu") (net 0))
-  (segment (start 111.712651 71.656741) (end 112.296406 71.55545) (width 0.25) (layer "F.Cu") (net 0))
-  (segment (start 105.532066 74.960333) (end 105.961166 74.551795) (width 0.25) (layer "F.Cu") (net 0))
-  (segment (start 108.906553 72.58375) (end 109.448202 72.343654) (width 0.25) (layer "F.Cu") (net 0))
-  (segment (start 131.9205 74.9371) (end 132.9111 75.9277) (width 0.25) (layer "F.Cu") (net 0))
+  (segment (start 110.563553 71.944575) (end 110.000979 72.130424) (width 0.25) (layer "F.Cu") (net 0))
+  (segment (start 131.267278 71.60857) (end 131.684664 71.831668) (width 0.25) (layer "F.Cu") (net 0))
+  (segment (start 112.884428 71.482924) (end 112.296406 71.55545) (width 0.25) (layer "F.Cu") (net 0))
+  (segment (start 132.050506 72.131906) (end 141.4926 81.574) (width 0.25) (layer "F.Cu") (net 0))
+  (segment (start 107.361273 73.45914) (end 106.876873 73.800294) (width 0.25) (layer "F.Cu") (net 0))
+  (segment (start 110.000979 72.130424) (end 109.448202 72.343654) (width 0.25) (layer "F.Cu") (net 0))
+  (segment (start 111.712651 71.656741) (end 111.134569 71.786554) (width 0.25) (layer "F.Cu") (net 0))
+  (segment (start 141.4926 81.574) (end 141.4926 84.5092) (width 0.25) (layer "F.Cu") (net 0))
+  (segment (start 130.814389 71.471188) (end 131.267278 71.60857) (width 0.25) (layer "F.Cu") (net 0))
+  (segment (start 106.409795 74.164805) (end 105.961166 74.551795) (width 0.25) (layer "F.Cu") (net 0))
+  (segment (start 108.377337 72.850135) (end 107.86183 73.142166) (width 0.25) (layer "F.Cu") (net 0))
+  (segment (start 114.0676 71.4248) (end 113.4753 71.439339) (width 0.25) (layer "F.Cu") (net 0))
+  (segment (start 108.906553 72.58375) (end 108.377337 72.850135) (width 0.25) (layer "F.Cu") (net 0))
+  (segment (start 141.478 84.5058) (end 141.478 84.4946) (width 0.25) (layer "F.Cu") (net 0))
+  (segment (start 113.4753 71.439339) (end 112.884428 71.482924) (width 0.25) (layer "F.Cu") (net 0))
+  (segment (start 130.3434 71.4248) (end 114.0676 71.4248) (width 0.25) (layer "F.Cu") (net 0))
+  (segment (start 109.448202 72.343654) (end 108.906553 72.58375) (width 0.25) (layer "F.Cu") (net 0))
+  (segment (start 106.876873 73.800294) (end 106.409795 74.164805) (width 0.25) (layer "F.Cu") (net 0))
   (segment (start 105.532066 74.960333) (end 98.6028 81.8896) (width 0.25) (layer "F.Cu") (net 0))
-  (segment (start 106.409795 74.164805) (end 106.876873 73.800294) (width 0.25) (layer "F.Cu") (net 0))
-  (segment (start 113.4753 71.439339) (end 114.0676 71.4248) (width 0.25) (layer "F.Cu") (net 0))
-  (segment (start 111.134569 71.786554) (end 111.712651 71.656741) (width 0.25) (layer "F.Cu") (net 0))
-  (segment (start 109.448202 72.343654) (end 110.000979 72.130424) (width 0.25) (layer "F.Cu") (net 0))
-  (segment (start 107.86183 73.142166) (end 108.377337 72.850135) (width 0.25) (layer "F.Cu") (net 0))
-  (segment (start 110.000979 72.130424) (end 110.563553 71.944575) (width 0.25) (layer "F.Cu") (net 0))
-  (segment (start 114.0676 71.4248) (end 128.4082 71.4248) (width 0.25) (layer "F.Cu") (net 0))
-  (segment (start 128.4082 71.4248) (end 131.9205 74.9371) (width 0.25) (layer "F.Cu") (net 0))
-  (segment (start 106.876873 73.800294) (end 107.361273 73.45914) (width 0.25) (layer "F.Cu") (net 0))
-  (segment (start 132.9111 75.9277) (end 141.4926 84.5092) (width 0.25) (layer "F.Cu") (net 0))
-  (segment (start 110.563553 71.944575) (end 111.134569 71.786554) (width 0.25) (layer "F.Cu") (net 0))
+  (segment (start 130.3434 71.4248) (end 130.814389 71.471188) (width 0.25) (layer "F.Cu") (net 0))
+  (segment (start 111.134569 71.786554) (end 110.563553 71.944575) (width 0.25) (layer "F.Cu") (net 0))
+  (segment (start 131.684664 71.831668) (end 132.050506 72.131906) (width 0.25) (layer "F.Cu") (net 0))
+  (segment (start 112.296406 71.55545) (end 111.712651 71.656741) (width 0.25) (layer "F.Cu") (net 0))
+  (segment (start 107.86183 73.142166) (end 107.361273 73.45914) (width 0.25) (layer "F.Cu") (net 0))
+  (segment (start 105.961166 74.551795) (end 105.532066 74.960333) (width 0.25) (layer "F.Cu") (net 0))
 )

Commit message: add 2 inch pumpkin
Parts:
- added Ref**: Val**, art:pumpkin25, F.Cu at (201.0, 117.5)
