File: pumpkin25.kicad_pcb (KiCad board)
At the start: 2 copper layers, 0 parts

Commit message: add 2 inch pumpkin
Parts:
- added Ref**: Val**, art:pumpkin25_, F.Cu at (-81.4, 232.0)
- added Ref**: Val**, art:pumpkin-outline-v3, F.Cu at (162.2, 80.1)
- added Ref**: Val**, art:pumpkin25cu, F.Cu at (166.5, 78.9)
- added Ref**: Val**, art:pumpkin25, F.Cu at (-28.8, 73.3)
- added Ref**: Val**, art:pumpkin25, F.Cu at (118.9, 132.7)
Other:
- board outline added: 89.3 x 76.4 mm
