File: art.kicad_pcb (KiCad board)
At the start: 2 copper layers, 43.2 x 43.2 mm, 2 parts

Commit message: update artwork
Parts:
- removed G*** (x2): LOGO, art:blm-1-5-inch-f-cu
- added REF**: PowerIntegrations_PDIP-8B, Package_DIP:PowerIntegrations_PDIP-8B, F.Cu at (132.2, 106.6)
Routing:
- added copper zone on F.Cu, net (none)
Other:
- board text added: "CU TEST"
- board text added: "MASK TEST"
- board text added: "SILK TEST"
