File: transistion46.kicad_pcb (KiCad board)
At the start: 2 copper layers, 29.8 x 29.8 mm, 2 parts

Commit message: update artwork
Parts:
- added Ref**: Val**, art:potus46, B.Cu at (138.9, 93.0)
- added Ref**: Val**, art:potus46-mask, B.Cu at (138.9, 93.0)
