File: keychain-blm-1_5-round.kicad_pcb (KiCad board)
At the start: 2 copper layers, 40.7 x 46.7 mm, 2 parts

Commit message: update artwork
Parts:
- added REF**: DTF13-12Px, Connector:DTF13-12Px, F.Cu at (191.5, 83.1)
Routing:
- net (no net): track 0.00 -> 90.2 mm, vias 1 -> 3
Changed lines of the file:
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@@
       (xy -5.103817 -15.660051)) (layer "F.Cu") (width 0))
+  )
+  (module "Connector:DTF13-12Px" (layer "F.Cu")
+    (at 191.4906 83.0834)
+    (descr "http://www.te.com/usa-en/product-DTF13-12PA-G003.html")
+    (tags "DEUTSCH DT header 12 pin ")
+    (attr through_hole)
+    (fp_text reference "REF**" (at 12.192 -3.81) (layer "F.SilkS")
+      (effects (font (size 1 1) (thickness 0.15)))
+    )
+    (fp_text value "DTF13-12Px" (at 11.6 23.1) (layer "F.Fab")
+      (effects (font (size 1 1) (thickness 0.15)))
+    )
+    (fp_text user "${REFERENCE}" (at 11.7 18.9) (layer "F.Fab")
+      (effects (font (size 1 1) (thickness 0.15)))
+    )
+    (fp_line (start -4.3434 5.588) (end -6.0198 5.588) (layer "F.SilkS") (width 0.15))
+    (fp_line (start 26.5684 5.588) (end 26.5684 12.7508) (layer "F.SilkS") (width 0.15))
+    (fp_line (start -4.3434 -2.1082) (end 26.5684 -2.1082) (layer "F.SilkS") (width 0.15))
+    (fp_line (start -4.3434 32.5882) (end -4.3688 27.9146) (layer "F.SilkS") (width 0.15))
+    (fp_line (start 26.5684 -1.1684) (end 26.5684 -2.1082) (layer "F.SilkS") (width 0.15))
+    (fp_line (start 28.2956 -1.1684) (end 26.5684 -1.1684) (layer "F.SilkS") (width 0.15))
+    (fp_line (start 28.9052 27.9146) (end 28.9052 12.7508) (layer "F.SilkS") (width 0.15))
+    (fp_line (start -6.0198 -1.1684) (end -4.3434 -1.1684) (layer "F.SilkS") (width 0.15))
+    (fp_line (start -6.6802 12.7508) (end -4.3434 12.7508) (layer "F.SilkS") (width 0.15))
+    (fp_line (start -6.6802 27.9146) (end -6.6802 12.7508) (layer "F.SilkS") (width 0.15))
+    (fp_line (start 26.5938 32.5882) (end -4.3434 32.5882) (layer "F.SilkS") (width 0.15))
+    (fp_line (start 26.5684 12.7508) (end 28.9052 12.7508) (layer "F.SilkS") (width 0.15))
+    (fp_line (start -4.3434 -1.1684) (end -4.3434 -2.1082) (layer "F.SilkS") (width 0.15))
+    (fp_line (start -4.3688 27.9146) (end -6.6802 27.9146) (layer "F.SilkS") (width 0.15))
+    (fp_line (start 26.5684 27.9146) (end 26.5938 32.5882) (layer "F.SilkS") (width 0.15))
+    (fp_line (start 28.9052 27.9146) (end 26.5684 27.9146) (layer "F.SilkS") (width 0.15))
+    (fp_line (start 28.2956 5.588) (end 26.5684 5.588) (layer "F.SilkS") (width 0.15))
+    (fp_line (start -4.3434 12.7508) (end -4.3434 5.588) (layer "F.SilkS") (width 0.15))
+    (fp_arc (start -6.0325 2.2098) (end -6.0325 5.588) (angle 180) (layer "F.SilkS") (width 0.15))
+    (fp_arc (start 28.321 2.2098) (end 28.321 5.588) (angle -180) (layer "F.SilkS") (width 0.15))
+    (fp_line (start -9.71 -1.46) (end -4.63 -1.46) (layer "F.CrtYd") (width 0.05))
+    (fp_line (start -9.71 5.88) (end -9.71 -1.46) (layer "F.CrtYd") (width 0.05))
+    (fp_line (start -9.71 5.88) (end -4.63 5.88) (layer "F.CrtYd") (width 0.05))
+    (fp_line (start 26.85 5.88) (end 31.94 5.88) (layer "F.CrtYd") (width 0.05))
+    (fp_line (start 26.85 28.19) (end 29.2 28.19) (layer "F.CrtYd") (width 0.05))
+    (fp_line (start 26.85 28.19) (end 26.85 32.88) (layer "F.CrtYd") (width 0.05))
+    (fp_line (start -4.63 32.88) (end -4.63 28.19) (layer "F.CrtYd") (width 0.05))
+    (fp_line (start -4.63 32.88) (end 26.85 32.88) (layer "F.CrtYd") (width 0.05))
+    (fp_line (start -4.63 12.45) (end -4.63 5.88) (layer "F.CrtYd") (width 0.05))
+    (fp_line (start -4.63 -1.46) (end -4.63 -2.4) (layer "F.CrtYd") (width 0.05))
+    (fp_line (start -6.98 28.19) (end -6.98 12.45) (layer "F.CrtYd") (width 0.05))
+    (fp_line (start 31.94 -1.47) (end 31.94 5.88) (layer "F.CrtYd") (width 0.05))
+    (fp_line (start -6.98 12.45) (end -4.63 12.45) (layer "F.CrtYd") (width 0.05))
+    (fp_line (start -6.98 28.19) (end -4.63 28.19) (layer "F.CrtYd") (width 0.05))
+    (fp_line (start 26.85 5.88) (end 26.85 12.45) (layer "F.CrtYd") (width 0.05))
+    (fp_line (start -4.63 -2.4) (end 26.85 -2.4) (layer "F.CrtYd") (width 0.05))
+    (fp_line (start 26.85 12.45) (end 29.2 12.45) (layer "F.CrtYd") (width 0.05))
+    (fp_line (start 26.85 -1.47) (end 31.94 -1.47) (layer "F.CrtYd") (width 0.05))
+    (fp_line (start 26.85 -1.47) (end 26.85 -2.4) (layer "F.CrtYd") (width 0.05))
+    (fp_line (start 29.2 12.45) (end 29.2 28.19) (layer "F.CrtYd") (width 0.05))
+    (fp_line (start 28.2575 5.3848) (end 26.3525 5.3848) (layer "F.Fab") (width 0.12))
+    (fp_line (start 26.3525 12.954) (end 28.702 12.954) (layer "F.Fab") (width 0.12))
+    (fp_line (start -4.1275 -1.905) (end -4.1275 32.385) (layer "F.Fab") (width 0.12))
+    (fp_line (start -0.635 -1.905) (end -4.1275 -1.905) (layer "F.Fab") (width 0.12))
+    (fp_line (start -0.635 6.35) (end -4.1275 6.35) (layer "F.Fab") (width 0.12))
+    (fp_line (start 26.3525 32.385) (end -4.1275 32.385) (layer "F.Fab") (width 0.12))
+    (fp_line (start -6.0325 5.3848) (end -4.1275 5.3848) (layer "F.Fab") (width 0.12))
+    (fp_line (start 28.2575 -0.9652) (end 26.3525 -0.9652) (layer "F.Fab") (width 0.12))
+    (fp_line (start -6.0325 -0.9652) (end -4.1275 -0.9652) (layer "F.Fab") (width 0.12))
+    (fp_line (start -0.635 -1.905) (end -0.635 6.35) (layer "F.Fab") (width 0.12))
+    (fp_line (start -6.477 27.686) (end -4.1275 27.686) (layer "F.Fab") (width 0.12))
+    (fp_line (start -6.477 12.954) (end -6.477 27.686) (layer "F.Fab") (width 0.12))
+    (fp_line (start -0.635 6.35) (end 22.86 6.35) (layer "F.Fab") (width 0.12))
+    (fp_line (start 22.86 -1.905) (end 26.3525 -1.905) (layer "F.Fab") (width 0.12))
+    (fp_line (start 28.702 27.686) (end 26.3525 27.686) (layer "F.Fab") (width 0.12))
+    (fp_line (start -4.1275 12.954) (end -6.477 12.954) (layer "F.Fab") (width 0.12))
+    (fp_line (start 22.86 -1.905) (end 22.86 6.35) (layer "F.Fab") (width 0.12))
+    (fp_line (start 28.702 12.954) (end 28.702 27.686) (layer "F.Fab") (width 0.12))
+    (fp_line (start -0.635 -1.905) (end 22.86 -1.905) (layer "F.Fab") (width 0.12))
+    (fp_line (start 22.86 6.35) (end 26.3525 6.35) (layer "F.Fab") (width 0.12))
+    (fp_line (start 26.3525 -1.905) (end 26.3525 32.385) (layer "F.Fab") (width 0.12))
+    (fp_arc (start -6.0325 2.2098) (end -6.0325 5.3848) (angle 180.6) (layer "F.Fab") (width 0.12))
+    (fp_arc (start 28.2575 2.2098) (end 28.2575 5.3848) (angle -180) (layer "F.Fab") (width 0.12))
+    (pad "" np_thru_hole circle (at 28.2575 2.2098) (size 2.4 2.4) (drill 2.4) (layers *.Cu *.Mask))
+    (pad "" np_thru_hole circle (at -6.0325 2.2098) (size 2.4 2.4) (drill 2.4) (layers *.Cu *.Mask))
+    (pad "1" thru_hole rect (at 0 0) (size 3 3) (drill 1.75) (layers *.Cu *.Mask))
+    (pad "2" thru_hole circle (at 4.445 0) (size 3 3) (drill 1.75) (layers *.Cu *.Mask))
+    (pad "3" thru_hole circle (at 8.89 0) (size 3 3) (drill 1.75) (layers *.Cu *.Mask))
+    (pad "4" thru_hole circle (at 13.335 0) (size 3 3) (drill 1.75) (layers *.Cu *.Mask))
+    (pad "5" thru_hole circle (at 17.78 0) (size 3 3) (drill 1.75) (layers *.Cu *.Mask))
+    (pad "6" thru_hole circle (at 22.225 0) (size 3 3) (drill 1.75) (layers *.Cu *.Mask))
+    (pad "7" thru_hole circle (at 22.225 4.445) (size 3 3) (drill 1.75) (layers *.Cu *.Mask))
+    (pad "8" thru_hole circle (at 17.78 4.445) (size 3 3) (drill 1.75) (layers *.Cu *.Mask))
+    (pad "9" thru_hole circle (at 13.335 4.445) (size 3 3) (drill 1.75) (layers *.Cu *.Mask))
+    (pad "10" thru_hole circle (at 8.89 4.445) (size 3 3) (drill 1.75) (layers *.Cu *.Mask))
+    (pad "11" thru_hole circle (at 4.445 4.445) (size 3 3) (drill 1.75) (layers *.Cu *.Mask))
+    (pad "12" thru_hole circle (at 0 4.445) (size 3.556 3.556) (drill 1.75) (layers *.Cu *.Mask))
+    (model "${KISYS3DMOD}/Connector.3dshapes/DTF13-12Px.wrl"
+      (offset (xyz 0 0 0))
+      (scale (xyz 1 1 1))
+      (rotate (xyz 0 0 0))
+    )
   )
   (module "art:blm-1-5-inch-f-cu" (layer "B.Cu")
@@
   )
   (gr_poly (pts
+ (xy 170.8404 67.0052)
+    (xy 172.0088 125.3236)
+    (xy 123.2662 124.8664)
+    (xy 125.2728 66.7004)
+    (xy 127.2794 66.548)) (layer "F.Mask") (width 0.1))
+  (gr_poly (pts
  (xy 167.5638 118.11)
     (xy 128.1938 118.11)
@@
   (gr_line (start 168.3766 86.36) (end 168.3766 118.1354) (layer "Edge.Cuts") (width 0.1))
   (gr_line (start 168.3766 80.2386) (end 168.3766 75.6158) (layer "Edge.Cuts") (width 0.1))
+  (segment (start 162.3314 78.3844) (end 164.6936 76.0222) (width 0.25) (layer "F.Cu") (net 0))
+  (segment (start 159.5882 78.3844) (end 162.3314 78.3844) (width 0.25) (layer "F.Cu") (net 0))
   (via (at 164.6936 76.0222) (size 5.588) (drill 5.08) (layers "F.Cu" "B.Cu") (net 0))
+  (via (at 159.5882 78.3844) (size 0.8) (drill 0.4) (layers "F.Cu" "B.Cu") (net 0))
+  (via (at 167.386 78.7654) (size 0.8) (drill 0.4) (layers "F.Cu" "B.Cu") (net 0))
+  (segment (start 195.9356 73.8886) (end 190.119 68.072) (width 0.25) (layer "B.Cu") (net 0))
+  (segment (start 172.6438 68.072) (end 164.6936 76.0222) (width 0.25) (layer "B.Cu") (net 0))
+  (segment (start 159.5882 78.3844) (end 160.2994 79.0956) (width 0.25) (layer "B.Cu") (net 0))
+  (segment (start 190.119 68.072) (end 172.6438 68.072) (width 0.25) (layer "B.Cu") (net 0))
+  (segment (start 171.7548 83.0834) (end 164.6936 76.0222) (width 0.25) (layer "B.Cu") (net 0))
+  (segment (start 160.2994 79.0956) (end 167.0558 79.0956) (width 0.25) (layer "B.Cu") (net 0))
+  (segment (start 191.4906 83.0834) (end 171.7548 83.0834) (width 0.25) (layer "B.Cu") (net 0))
+  (segment (start 195.9356 83.0834) (end 195.9356 73.8886) (width 0.25) (layer "B.Cu") (net 0))
+  (segment (start 167.0558 79.0956) (end 167.386 78.7654) (width 0.25) (layer "B.Cu") (net 0))
 )

Commit message: update
Parts:
- removed REF**: DTF13-12Px, Connector:DTF13-12Px
Routing:
- net (no net): track 90.2 -> 0.00 mm, vias 3 -> 1
