File: lauren.kicad_pcb (KiCad board)
At the start: 2 copper layers, 344.6 x 259.8 mm, 5 parts

Commit message: six layer artwork
Parts:
- removed the G*** at (146.7, -65.9) (x2)
- removed the G*** at (141.0, 97.3)
- removed the G*** at (141.8, 93.4)
- removed the G*** at (141.4, 97.4)
- added G***: LOGO, art:lauren-red-2-inch, F.Cu at (101.8, 28.8)
- added G***: LOGO, art:lauren-red-2-inch-cu, F.Cu at (101.8, 28.8)
- added G***: LOGO, art:lauren-red-2-inch, F.Cu at (119.4, 74.6)
Other:
- board size 344.6 x 259.8 mm -> 127.9 x 127.9 mm
