File: art2.kicad_pcb (KiCad board)
At the start: 2 copper layers, 4.6 x 4.6 mm, 0 parts

Commit message: update
Routing:
- added copper zone on F.Cu, net (none)
Other:
- board size 4.6 x 4.6 mm -> 106.9 x 65.2 mm
Changed lines of the file:
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@@
-(kicad_pcb (version 20200922) (generator pcbnew)
+(kicad_pcb (version 20201220) (generator pcbnew)
   (general
     (thickness 1.6)
@@
     (pcbplotparams
       (layerselection 0x00010fc_ffffffff)
+      (disableapertmacros false)
       (usegerberextensions false)
       (usegerberattributes true)
@@
       (svgprecision 6)
       (excludeedgelayer true)
-      (linewidth 0.100000)
       (plotframeref false)
       (viasonmask false)
@@
       (hpglpenspeed 20)
       (hpglpendiameter 15.000000)
+      (dxfpolygonmode true)
+      (dxfimperialunits true)
+      (dxfusepcbnewfont true)
       (psnegative false)
       (psa4output false)
@@
   )
   (net 0 "")
-  (gr_line (start 41.7576 156.1338) (end 43.18 156.1338) (layer "F.Cu") (width 0.2))
-  (gr_line (start 43.18 156.1338) (end 44.2722 157.226) (layer "F.Cu") (width 0.2))
-  (gr_rect (start 40.132 154.432) (end 44.704 159.004) (layer "Edge.Cuts") (width 0.05))
+  (gr_rect (start 142.7988 146.2024) (end 35.9156 81.0006) (layer "Edge.Cuts") (width 0.05) (fill none))
+  (zone (net 0) (net_name "") (layer "F.Cu") (hatch edge 0.508)
+    (connect_pads (clearance 0.508))
+    (min_thickness 0.254) (filled_areas_thickness no)
+    (fill yes (thermal_gap 0.508) (thermal_bridge_width 0.508))
+    (polygon
+      (pts
+        (xy 132.08 142.9258)
+        (xy 40.132 142.9258)
+        (xy 40.132 83.439)
+        (xy 132.08 83.439)
+      )
+    )
+  )
 )
