File: flower-v3.kicad_pcb (KiCad board)
At the start: 2 copper layers, 25.9 x 52.8 mm, 7 parts

Commit message: update
Parts:
- removed PG4: CONN_01X01, hex-smd-challenge-fp:testPad
- REF**: value 1206 -> 0805; footprint digikey-footprints:1206 -> digikey-footprints:0805
Routing:
- net (no net): track 81.3 -> 80.5 mm
Other:
- board text removed: "`"
Changed lines of the file:
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@@
     (34 "B.Paste" user)
     (35 "F.Paste" user)
-    (36 "B.SilkS" user "B.Silkscreen")
-    (37 "F.SilkS" user "F.Silkscreen")
+    (36 "B.SilkS" user)
+    (37 "F.SilkS" user)
     (38 "B.Mask" user)
     (39 "F.Mask" user)
@@
       (drillshape 0)
       (scaleselection 1)
-      (outputdirectory "gerbers/flower")
+      (outputdirectory "gerbers/flower-v3")
     )
   )
@@
     (pad "1" smd roundrect (at -0.3556 1.143 90) (size 2.54 3.302) (layers "B.Cu" "B.Mask") (roundrect_rratio 0.2))
   )
-  (footprint "hex-smd-challenge-fp:testPad" (layer "B.Cu")
-    (at 62.4332 38.5826)
-    (descr "module 1 pin (ou trou mecanique de percage)")
-    (tags "DEV")
-    (attr through_hole)
-    (fp_text reference "PG4" (at -0.0635 0) (layer "B.SilkS") hide
-      (effects (font (size 0.635 0.635) (thickness 0.127)) (justify mirror))
-    )
-    (fp_text value "CONN_01X01" (at 0 0) (layer "B.Fab")
-      (effects (font (size 0.127 0.127) (thickness 0.03175)) (justify mirror))
-    )
-    (pad "1" smd oval (at 0 0 270) (locked) (size 1 2) (layers "B.Cu" "B.Paste" "B.Mask"))
-  )
-  (footprint "digikey-footprints:1206" (layer "B.Cu")
+  (footprint "digikey-footprints:0805" (layer "B.Cu")
     (at 62.5 35.5)
-    (descr "http://media.digikey.com/pdf/Data%20Sheets/Lite-On%20PDFs/LTST-C230KFKT_5-24-06.pdf")
     (attr smd)
-    (fp_text reference "REF**" (at 0.1 2.5) (layer "B.SilkS") hide
+    (fp_text reference "REF**" (at 0 1.84) (layer "B.SilkS")
       (effects (font (size 1 1) (thickness 0.15)) (justify mirror))
     )
-    (fp_text value "1206" (at 0 -2.6) (layer "B.Fab") hide
+    (fp_text value "0805" (at 0 -1.95) (layer "B.Fab")
       (effects (font (size 1 1) (thickness 0.15)) (justify mirror))
     )
@@
       (effects (font (size 1 1) (thickness 0.15)) (justify mirror))
     )
-    (fp_line (start 2.8 -1.15) (end 2.8 1.15) (layer "B.CrtYd") (width 0.05))
-    (fp_line (start -2.8 -1.15) (end 2.8 -1.15) (layer "B.CrtYd") (width 0.05))
-    (fp_line (start -2.8 1.15) (end -2.8 -1.15) (layer "B.CrtYd") (width 0.05))
-    (fp_line (start 2.8 1.15) (end -2.8 1.15) (layer "B.CrtYd") (width 0.05))
-    (fp_line (start -1.6 0.8) (end -1.6 -0.8) (layer "B.Fab") (width 0.1))
-    (fp_line (start 1.6 0.8) (end 1.6 -0.8) (layer "B.Fab") (width 0.1))
-    (pad "1" smd roundrect (at -1.8 0) (locked) (size 1.5 1.8) (layers "B.Cu" "B.Paste" "B.Mask") (roundrect_rratio 0.25))
-    (pad "2" smd roundrect (at 1.8 0) (locked) (size 1.5 1.8) (layers "B.Cu" "B.Paste" "B.Mask") (roundrect_rratio 0.25))
-  )
-  (gr_circle (center 62.3316 35.6362) (end 67.5132 35.6108) (layer "F.Cu") (width 0.2) (fill solid))
+    (fp_line (start -0.32 -0.8) (end 0.28 -0.8) (layer "B.SilkS") (width 0.12))
+    (fp_line (start -0.3 0.8) (end 0.3 0.8) (layer "B.SilkS") (width 0.12))
+    (fp_line (start -1.9 -0.93) (end -1.9 0.93) (layer "B.CrtYd") (width 0.05))
+    (fp_line (start -1.9 0.93) (end 1.9 0.93) (layer "B.CrtYd") (width 0.05))
+    (fp_line (start -1.9 -0.93) (end 1.9 -0.93) (layer "B.CrtYd") (width 0.05))
+    (fp_line (start 1.9 -0.93) (end 1.9 0.93) (layer "B.CrtYd") (width 0.05))
+    (fp_line (start 0.95 0.675) (end 0.95 -0.675) (layer "B.Fab") (width 0.12))
+    (fp_line (start -0.95 0.675) (end -0.95 -0.675) (layer "B.Fab") (width 0.12))
+    (fp_line (start -0.95 -0.68) (end 0.95 -0.68) (layer "B.Fab") (width 0.12))
+    (fp_line (start -0.95 0.68) (end 0.95 0.68) (layer "B.Fab") (width 0.12))
+    (pad "1" smd rect (at -1.05 0) (locked) (size 1.2 1.2) (layers "B.Cu" "B.Paste" "B.Mask"))
+    (pad "2" smd rect (at 1.05 0) (locked) (size 1.2 1.2) (layers "B.Cu" "B.Paste" "B.Mask"))
+  )
   (gr_circle (center 62.357 35.642289) (end 67.437 35.642289) (layer "B.SilkS") (width 0.12) (fill solid))
-  (gr_circle (center 62.3316 35.6362) (end 66.8528 35.433) (layer "F.Mask") (width 0.2) (fill solid))
+  (gr_circle (center 62.3316 35.6362) (end 67.513262 35.6362) (layer "F.SilkS") (width 0.2) (fill solid))
   (gr_text "Happy" (at 56.5658 59.7154 325) (layer "F.Cu")
     (effects (font (size 1.5 1.5) (thickness 0.3)))
@@
     (effects (font (size 1.5 1.5) (thickness 0.3)))
   )
-  (gr_text "`" (at 60.7314 34.417) (layer "B.Mask")
-    (effects (font (size 1 1) (thickness 0.15)) (justify mirror))
-  )
-  (gr_text "`" (at 64.3382 34.4424) (layer "B.Mask")
-    (effects (font (size 1 1) (thickness 0.15)) (justify mirror))
-  )
   (via (at 66.8528 72.898) (size 1.27) (drill 0.762) (layers "F.Cu" "B.Cu") (net 0))
   (via (at 60.3504 72.898) (size 1.27) (drill 0.762) (layers "F.Cu" "B.Cu") (net 0))
-  (segment (start 63.3476 55.208331) (end 63.3476 59.199432) (width 0.25) (layer "B.Cu") (net 0))
-  (segment (start 63.3476 59.199432) (end 63.7286 60.119247) (width 0.25) (layer "B.Cu") (net 0))
-  (segment (start 64.0842 71.628) (end 65.3542 72.898) (width 0.25) (layer "B.Cu") (net 0))
-  (segment (start 62.9412 60.485368) (end 62.9412 68.9356) (width 0.25) (layer "B.Cu") (net 0))
-  (segment (start 64.3 35.5) (end 64.3 37.533009) (width 0.25) (layer "B.Cu") (net 0))
-  (segment (start 60.7 35.5) (end 60.7 38.160348) (width 0.25) (layer "B.Cu") (net 0))
-  (segment (start 63.2206 72.517) (end 62.7888 72.9488) (width 0.25) (layer "B.Cu") (net 0))
-  (segment (start 62.667484 59.920717) (end 62.738 59.9948) (width 0.25) (layer "B.Cu") (net 0))
-  (segment (start 65.3542 72.898) (end 66.8528 72.898) (width 0.25) (layer "B.Cu") (net 0))
-  (segment (start 62.0776 41.486168) (end 62.0776 54.40319) (width 0.25) (layer "B.Cu") (net 0))
-  (segment (start 61.736843 40.854745) (end 61.8744 40.9956) (width 0.25) (layer "B.Cu") (net 0))
-  (segment (start 63.2206 69.215) (end 63.2206 72.517) (width 0.25) (layer "B.Cu") (net 0))
-  (segment (start 64.0842 68.7832) (end 64.0842 71.628) (width 0.25) (layer "B.Cu") (net 0))
-  (segment (start 64.3 37.533009) (end 62.611 41.610615) (width 0.25) (layer "B.Cu") (net 0))
-  (segment (start 63.7286 60.119247) (end 63.7286 68.4276) (width 0.25) (layer "B.Cu") (net 0))
-  (segment (start 62.9412 68.9356) (end 63.2206 69.215) (width 0.25) (layer "B.Cu") (net 0))
-  (segment (start 63.7286 68.4276) (end 64.0842 68.7832) (width 0.25) (layer "B.Cu") (net 0))
-  (segment (start 62.7888 72.9488) (end 60.325 72.9488) (width 0.25) (layer "B.Cu") (net 0))
+  (segment (start 61.45 38.226376) (end 61.45 35.5) (width 0.25) (layer "B.Cu") (net 0))
+  (segment (start 63.045434 38.381181) (end 63.1444 38.2778) (width 0.25) (layer "B.Cu") (net 0))
+  (segment (start 61.747056 38.83878) (end 61.6712 38.7604) (width 0.25) (layer "B.Cu") (net 0))
+  (segment (start 62.0776 54.40319) (end 62.0776 39.741536) (width 0.25) (layer "B.Cu") (net 0))
+  (segment (start 63.2206 72.517) (end 62.7888 72.9488) (width 0.508) (layer "B.Cu") (net 0))
+  (segment (start 63.3476 59.199432) (end 63.3476 55.208331) (width 0.25) (layer "B.Cu") (net 0))
+  (segment (start 62.4332 60.198) (end 62.4332 55.261684) (width 0.25) (layer "B.Cu") (net 0))
+  (segment (start 64.2112 68.8848) (end 63.7286 61.7982) (width 0.25) (layer "B.Cu") (net 0))
+  (segment (start 63.2206 69.215) (end 63.2206 72.517) (width 0.508) (layer "B.Cu") (net 0))
+  (segment (start 63.7286 60.119247) (end 63.3476 59.199432) (width 0.25) (layer "B.Cu") (net 0))
+  (segment (start 64.4652 72.3392) (end 64.2112 68.8848) (width 0.508) (layer "B.Cu") (net 0))
+  (segment (start 63.2206 69.215) (end 62.4332 60.198) (width 0.25) (layer "B.Cu") (net 0))
+  (segment (start 62.7888 72.9488) (end 60.325 72.9488) (width 0.508) (layer "B.Cu") (net 0))
   (segment (start 62.272515 54.954928) (end 62.3316 55.0164) (width 0.25) (layer "B.Cu") (net 0))
-  (segment (start 62.4332 55.261684) (end 62.4332 59.258948) (width 0.25) (layer "B.Cu") (net 0))
-  (segment (start 62.611 41.610615) (end 62.611 53.430022) (width 0.25) (layer "B.Cu") (net 0))
-  (segment (start 62.611 53.430022) (end 63.3476 55.208331) (width 0.25) (layer "B.Cu") (net 0))
-  (arc (start 60.7 38.160348) (mid 61.005215 39.694775) (end 61.8744 40.9956) (width 0.25) (layer "B.Cu") (net 0))
-  (arc (start 62.0776 54.40319) (mid 62.143611 54.735056) (end 62.3316 55.0164) (width 0.25) (layer "B.Cu") (net 0))
-  (arc (start 62.3316 55.0164) (mid 62.406794 55.128936) (end 62.4332 55.261684) (width 0.25) (layer "B.Cu") (net 0))
-  (arc (start 62.4332 59.258948) (mid 62.512414 59.657188) (end 62.738 59.9948) (width 0.25) (layer "B.Cu") (net 0))
-  (arc (start 62.738 59.9948) (mid 62.888389 60.219874) (end 62.9412 60.485368) (width 0.25) (layer "B.Cu") (net 0))
-  (arc (start 61.8744 40.9956) (mid 62.024789 41.220674) (end 62.0776 41.486168) (width 0.25) (layer "B.Cu") (net 0))
+  (segment (start 63.3476 55.208331) (end 62.611 39.565541) (width 0.25) (layer "B.Cu") (net 0))
+  (segment (start 66.8528 72.898) (end 65.3542 72.898) (width 0.508) (layer "B.Cu") (net 0))
+  (segment (start 65.3542 72.898) (end 64.4652 72.3392) (width 0.508) (layer "B.Cu") (net 0))
+  (segment (start 63.7286 61.7982) (end 63.7286 60.119247) (width 0.25) (layer "B.Cu") (net 0))
+  (segment (start 63.55 37.298595) (end 63.55 35.5) (width 0.25) (layer "B.Cu") (net 0))
+  (arc (start 62.0776 39.741536) (mid 61.97198 39.210549) (end 61.6712 38.7604) (width 0.25) (layer "B.Cu") (net 0))
+  (arc (start 62.3316 55.0164) (mid 62.143611 54.735056) (end 62.0776 54.40319) (width 0.25) (layer "B.Cu") (net 0))
+  (arc (start 63.1444 38.2778) (mid 63.444588 37.828538) (end 63.55 37.298595) (width 0.25) (layer "B.Cu") (net 0))
+  (arc (start 62.611 39.565541) (mid 62.749626 38.868621) (end 63.1444 38.2778) (width 0.25) (layer "B.Cu") (net 0))
+  (arc (start 62.4332 55.261684) (mid 62.406794 55.128936) (end 62.3316 55.0164) (width 0.25) (layer "B.Cu") (net 0))
+  (arc (start 61.6712 38.7604) (mid 61.507488 38.515389) (end 61.45 38.226376) (width 0.25) (layer "B.Cu") (net 0))
   (zone (net 0) (net_name "") (layer "F.Cu") (hatch edge 0.508)
     (connect_pads (clearance 0.0254))
