File: cutouts/cutouts.kicad_pcb (KiCad board)
At the start: 2 copper layers, 25.4 x 25.4 mm, 0 parts

Commit message: add cutout tests
Parts:
- added REF**: drag drill, MountingHole:MountingHole_2.5mm_Pad, F.Cu at (148.9, 64.9)
Routing:
- net (no net): vias 1 -> 0
Changed lines of the file:
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@@
     (34 "B.Paste" user)
     (35 "F.Paste" user)
-    (36 "B.SilkS" user)
-    (37 "F.SilkS" user)
+    (36 "B.SilkS" user "B.Silkscreen")
+    (37 "F.SilkS" user "F.Silkscreen")
     (38 "B.Mask" user)
     (39 "F.Mask" user)
@@
   )
   (net 0 "")
+  (footprint "MountingHole:MountingHole_2.5mm_Pad" (layer "F.Cu")
+    (at 148.9456 64.8716)
+    (descr "Mounting Hole 2.5mm")
+    (tags "mounting hole 2.5mm")
+    (attr exclude_from_pos_files exclude_from_bom)
+    (fp_text reference "REF**" (at 0 -3.5) (layer "F.SilkS") hide
+      (effects (font (size 1 1) (thickness 0.15)))
+    )
+    (fp_text value "drag drill" (at 0 3.5) (layer "F.Fab") hide
+      (effects (font (size 1 1) (thickness 0.15)))
+    )
+    (pad "1" thru_hole oval (at 0 0) (size 2.286 0.762) (drill oval 2.032 0.508) (layers *.Cu *.Mask))
+  )
   (gr_line (start 128.4986 62.103) (end 128.4986 87.4268) (layer "Eco2.User") (width 0.15))
   (gr_line (start 142.621 62.1284) (end 142.621 87.4522) (layer "Eco2.User") (width 0.15))
@@
     (effects (font (size 1 1) (thickness 0.15)))
   )
-  (via (at 149.479 63.9318) (size 1.778) (drill 1.524) (layers "F.Cu" "B.Cu") (free) (net 0))
 )
